Commit message: added arm to main bot

File: install/my_robot_description/share/my_robot_description/urdf/camera.xacro (robot description, xacro)
@@ -1,37 +1 @@
-<?xml version = "1.0"?>
-<robot name="my_robot" xmlns:xacro="http://www.ros.org/wiki/xacro">
-    <xacro:property name="camera_length" value="0.01" />
-    <xacro:property name="camera_width" value="0.1" />
-    <xacro:property name="camera_height" value="0.05" />
-    <link name="camera_link">
-        <visual>
-            <geometry>
-                <box size="${camera_length} ${camera_width} ${camera_height}" />
-            </geometry>
-            <material name="grey" />
-        </visual>
-        <collision>
-            <geometry>
-                <box size="${camera_length} ${camera_width} ${camera_height}" />
-            </geometry>
-        </collision>
-        <xacro:box_inertia m="0.1" l="${camera_length}" w="${camera_width}" h="${camera_height}"
-                           xyz="0 0 0" rpy="0 0 0" />
-    </link>
-    <joint name="base_camera_joint" type="fixed">
-        <parent link="base_link" />
-        <child link="camera_link" />
-        <origin xyz="${(base_length + camera_length) / 2} 0 ${base_height / 2}" rpy="0 0 0" />
-    </joint>
-    <gazebo reference="camera_link">
-        <material>Gazebo/Red</material>
-        <sensor name="camera_sensor" type="camera">
-            <pose>0 0 0 0 0 0</pose>
-            <visualize>true</visualize>
-            <update_rate>10.0</update_rate>
-            <plugin name="camera_controller" filename="libgazebo_ros_camera.so">
-                <frame_name>camera_link</frame_name>
-            </plugin>
-        </sensor>
-    </gazebo>
-</robot>
+/home/sambhav/ros2_ws/src/my_robot_description/urdf/camera.xacro

File: install/my_robot_description/share/my_robot_description/urdf/common_properties.xacro (robot description, xacro)
@@ -1,36 +1 @@
-<?xml version = "1.0"?>
-<robot xmlns:xacro="http://www.ros.org/wiki/xacro">
-    <material name="green">
-        <color rgba="0 0.5 0 1" />
-    </material>
-    <material name="grey">
-        <color rgba="0.5 0.5 0.5 1" />
-    </material>
-    <xacro:macro name="box_inertia" params="m l w h xyz rpy">
-        <inertial>
-            <origin xyz="${xyz}" rpy="${rpy}" />
-            <mass value="${m}" />
-            <inertia ixx="${(m/12.0) * (h*h + l*l)}" ixy="0" ixz="0"
-                     iyy="${(m/12.0) * (w*w + l*l)}" iyz="0"
-                     izz="${(m/12.0) * (w*w + h*h)}" />
-        </inertial>
-    </xacro:macro>
-    <xacro:macro name="sphere_inertia" params="m r xyz rpy">
-        <inertial>
-            <origin xyz="${xyz}" rpy="${rpy}" />
-            <mass value="${m}" />
-            <inertia ixx="${(m * 2.0/5.0) * (r*r)}" ixy="0" ixz="0"
-                     iyy="${(m * 2.0/5.0) * (r*r)}"  iyz="0"
-                     izz="${(m * 2.0/5.0) * (r*r)}" />
-        </inertial>
-    </xacro:macro>
-    <xacro:macro name="cylinder_inertia" params="m r h xyz rpy">
-        <inertial>
-            <origin xyz="${xyz}" rpy="${rpy}" />
-            <mass value="${m}" />
-            <inertia ixx="${(m/12) * (3*r*r + h*h)}" ixy="0" ixz="0"
-                     iyy="${(m/12) * (3*r*r + h*h)}" iyz="0"
-                     izz="${(m/12) * (3*r*r + h*h)}" />
-        </inertial>
-    </xacro:macro>
-</robot>
+/home/sambhav/ros2_ws/src/my_robot_description/urdf/common_properties.xacro

File: install/my_robot_description/share/my_robot_description/urdf/mobile_base.xacro (robot description, xacro)
@@ -1,86 +1 @@
-<?xml version = "1.0"?>
-<robot xmlns:xacro="http://www.ros.org/wiki/xacro">
-    <xacro:property name="base_length" value="0.6" />
-    <xacro:property name="base_width" value="0.4" />
-    <xacro:property name="base_height" value="0.2" />
-    <xacro:property name="wheel_radius" value="0.1" />
-    <xacro:property name="wheel_length" value="0.05" />
-    <link name="base_footprint" />
-    <link name="base_link">
-        <visual>
-            <geometry>
-                <box size="${base_length} ${base_width} ${base_height}" />
-            </geometry>
-            <origin xyz="0 0 ${base_height / 2.0}" rpy="0 0 0" />
-            <material name="green" />
-        </visual>
-        <collision>
-            <geometry>
-                <box size="${base_length} ${base_width} ${base_height}" />
-            </geometry>
-            <origin xyz="0 0 ${base_height / 2.0}" rpy="0 0 0" />
-        </collision>
-        <xacro:box_inertia m="5.0" l="${2*base_length}" w="${2*base_width}" h="${2*base_height}"
-                           xyz="0 0 ${base_height}" rpy="0 0 0" />
-    </link>
-    <xacro:macro name="wheel_link" params="prefix">
-        <link name="${prefix}_wheel_link">
-            <visual>
-                <geometry>
-                    <cylinder radius="${wheel_radius}" length="${wheel_length}" />
-                </geometry>
-                <origin xyz="0 0 0" rpy="${pi / 2.0} 0 0" />
-                <material name="grey" />
-            </visual>
-            <collision>
-                <geometry>
-                    <cylinder radius="${wheel_radius}" length="${wheel_length}" />
-                </geometry>
-                <origin xyz="0 0 0" rpy="${pi / 2.0} 0 0" />
-            </collision>
-            <xacro:cylinder_inertia m="1.0" r="${2*wheel_radius}" h="${2*wheel_length}"
-                           xyz="0 0 0" rpy="${pi / 2.0} 0 0" />
-        </link>
-    </xacro:macro>
-    <xacro:wheel_link prefix="right" />
-    <xacro:wheel_link prefix="left" />
-    <link name="caster_wheel_link">
-        <visual>
-            <geometry>
-                <sphere radius="${wheel_radius/2.0}"/>
-            </geometry>
-            <origin xyz="0 0 0" rpy="0 0 0" />
-            <material name="grey" />
-        </visual>
-        <collision>
-            <geometry>
-                <sphere radius="${wheel_radius/2.0}"/>
-            </geometry>
-            <origin xyz="0 0 0" rpy="0 0 0" />
-        </collision>
-        <xacro:sphere_inertia m="0.5" r="${2*wheel_radius / 2.0}"
-                           xyz="0 0 0" rpy="0 0 0" />
-    </link>
-    <joint name="base_joint" type="fixed">
-        <parent link="base_footprint" />
-        <child link="base_link" />
-        <origin xyz="0 0 0.1" rpy="0 0 0"/>
-    </joint>
-    <joint name="base_right_wheel_joint" type="continuous">
-        <parent link="base_link" />
-        <child link="right_wheel_link" />
-        <origin xyz="${-base_length / 4.0} ${(base_width / 2.0) + (wheel_length / 2.0)} 0" rpy="0 0 0" />
-        <axis xyz="0 1 0" />
-    </joint>
-    <joint name="base_left_wheel_joint" type="continuous">
-        <parent link="base_link" />
-        <child link="left_wheel_link" />
-        <origin xyz="${-base_length / 4.0} ${(-base_width / 2.0) + (-wheel_length / 2.0)} 0" rpy="0 0 0" />
-        <axis xyz="0 1 0" />
-    </joint>
-    <joint name="base_caster_wheel_joint" type="fixed">
-        <parent link="base_link" />
-        <child link="caster_wheel_link" />
-        <origin xyz="${base_length / 3.0} 0 ${-wheel_radius /2.0}" rpy="0 0 0" />
-    </joint>
-</robot>
+/home/sambhav/ros2_ws/src/my_robot_description/urdf/mobile_base.xacro

File: install/my_robot_description/share/my_robot_description/urdf/mobile_base_gazebo.xacro (robot description, xacro)
@@ -1,39 +1 @@
-<?xml version = "1.0"?>
-<robot xmlns:xacro="http://www.ros.org/wiki/xacro">
-    <gazebo reference="base_link">
-        <material>Gazebo/Blue</material>
-    </gazebo>
-    <gazebo reference="right_wheel_link">
-        <material>Gazebo/Grey</material>
-    </gazebo>
-    <gazebo reference="left_wheel_link">
-        <material>Gazebo/Grey</material>
-    </gazebo>
-    <gazebo reference="caster_wheel_link">
-        <material>Gazebo/Grey</material>
-        <mu1 value="0.1" />
-        <mu2 value="0.1" />
-    </gazebo>
-    <gazebo>
-        <plugin name="diff_drive_controller" filename="libgazebo_ros_diff_drive.so">
-            <!-- Update rate in Hz -->
-            <update_rate>50</update_rate>
-            <!-- wheels -->
-            <left_joint>base_left_wheel_joint</left_joint>
-            <right_joint>base_right_wheel_joint</right_joint>
-            <!-- kinematics -->
-            <wheel_separation>0.45</wheel_separation>
-            <wheel_diameter>0.2</wheel_diameter>
-            <!-- limits -->
-            <max_wheel_torque>20</max_wheel_torque>
-            <max_wheel_acceleration>1.0</max_wheel_acceleration>
-            <!-- output -->
-            <publish_odom>true</publish_odom>
-            <publish_odom_tf>true</publish_odom_tf>
-            <publish_wheel_tf>true</publish_wheel_tf>
-            <odometry_topic>odom</odometry_topic>
-            <odometry_frame>odom</odometry_frame>
-            <robot_base_frame>base_link</robot_base_frame>
-          </plugin>
-    </gazebo>
-</robot>
+/home/sambhav/ros2_ws/src/my_robot_description/urdf/mobile_base_gazebo.xacro

File: install/my_robot_description/share/my_robot_description/urdf/my_robot.urdf.xacro (robot description, xacro)
@@ -1,81 +1 @@
-<?xml version = "1.0"?>
-<robot name="my_robot" xmlns:xacro="http://www.ros.org/wiki/xacro">
-    <xacro:include filename="common_properties.xacro" />
-    <xacro:include filename="mobile_base.xacro" />
-    <xacro:include filename="mobile_base_gazebo.xacro" />
-    <xacro:include filename="camera.xacro" />
-</robot>
-    <!-- <link name="right_wheel_link">
-        <visual>
-            <geometry>
-                <cylinder radius="${wheel_radius}" length="${wheel_length}" />
-            </geometry>
-            <origin xyz="0 0 0" rpy="${pi / 2.0} 0 0" />
-            <material name="grey" />
-        </visual>
-    </link>
-    <link name="left_wheel_link">
-        <visual>
-            <geometry>
-                <cylinder radius="${wheel_radius}" length="${wheel_length}" />
-            </geometry>
-            <origin xyz="0 0 0" rpy="${pi / 2.0} 0 0" />
-            <material name="grey" />
-        </visual>
-    </link> -->
-    <!-- <xacro:macro name="example_macro" params="a b c">
-        <link name="dummy_link">
-            <visual>
-                <geometry>
-                    <box size="${a} ${b} ${c}" />
-                </geometry>
-            </visual>
-        </link>
-    </xacro:macro>
-    <xacro:example_macro a="2" b="3" c="4" /> -->
-    <!-- <link name="base_link">
-        <visual>
-            <geometry>
-                <box size="0.6 0.4 0.2" />
-            </geometry>
-            <origin xyz="0 0 0.1" rpy="0 0 0" />
-            <material name="green" />
-        </visual>
-    </link>
-    <link name="second_link">
-        <visual>
-            <geometry>
-                <cylinder radius="0.1" length="0.2" />
-            </geometry>
-            <origin xyz="0 0 0.1" rpy="0 0 0" />
-            <material name="grey" />
-        </visual>
-    </link>
-    <joint name="base_second_joint" type="prismatic">
-        <parent link="base_link" />
-        <child link="second_link" />
-        <origin xyz="0 0 0.2" rpy="0 0 0" />
-        <axis xyz="1 0 0"/>
-        <limit lower="0.0" upper="0.2" velocity="100" effort="100"/>
-    </joint>
-    <joint name="base_second_joint" type="revolute">
-        <parent link="base_link" />
-        <child link="second_link" />
-        <origin xyz="0 0 0.2" rpy="0 0 0" />
-        <axis xyz="0 0 1"/>
-        <limit lower="-1.57" upper="1.57" velocity="100" effort="100"/>
-    </joint>
-    <link name="third_link">
-        <visual>
-            <geometry>
-                <box size="0.1 0.1 0.1" />
-            </geometry>
-            <origin xyz="0 0 0.05" rpy="0 0 0" />
-            <material name="green" />
-        </visual>
-    </link>
-    <joint name="second_third_joint" type="fixed">
-        <parent link="second_link" />
-        <child link="third_link" />
-        <origin xyz="0 0 0.2" rpy="0 0 0" />
-    </joint> -->
+/home/sambhav/ros2_ws/src/my_robot_description/urdf/my_robot.urdf.xacro

File: install/my_robot_description/share/my_robot_description/urdf/robotic_arm.xacro (robot description, xacro)
@@ -1,74 +1 @@
-<?xml version = "1.0"?>
-<robot xmlns:xacro="http://www.ros.org/wiki/xacro">
-    <xacro:include filename="common_properties.xacro" />
-    <xacro:property name="forearm_length" value = "0.3" />
-    <xacro:property name="forearm_radius" value = "0.02" />
-    <xacro:property name="hand_length" value = "0.3" />
-    <xacro:property name="hand_radius" value = "0.02" />
-    <xacro:property name="box_length" value = "0.1" />
-    <xacro:property name="box_width" value = "0.1" />
-    <xacro:property name="box_height" value = "0.02" />
-    <link name = "base_footprint" />
-    <link name="box_link">
-        <visual>
-            <geometry>
-                <box size="${box_length} ${box_width} ${box_height}" />
-            </geometry>
-            <origin xyz="0 0 ${box_height/2.0}" rpy="0 0 0" />
-            <material name="green" />
-        </visual>
-        <collision>
-            <geometry>
-                <box size="${box_length} ${box_width} ${box_height}" />
-            </geometry>
-            <origin xyz="0 0 ${box_height/2.0}" rpy="0 0 0" />
-        </collision>
-        <xacro:box_inertia m="0.5" l="${2*box_length}" w="${2*box_width}" h="${2*box_height}"
-                           xyz="0 0 ${box_height}" rpy="0 0 0" />
-    </link>
-    <link name="forearm_link">
-        <visual>
-            <geometry>
-                <cylinder radius = "${forearm_radius}" length = "${forearm_length}" />
-            </geometry>
-            <origin xyz="0 0 0" rpy="0 0 0" />
-            <material name="green" />
-        </visual>
-        <collision>
-            <geometry>
-                <cylinder radius="${forearm_radius}" length="${forearm_length}" />
-            </geometry>
-            <origin xyz="0 0 0" rpy="0 0 0" />
-        </collision>
-        <xacro:cylinder_inertia m="1.0" r="${2*forearm_radius}" h="${2*forearm_length}"
-                       xyz="0 0 0" rpy="$0 0 0" />
-    </link>
-    <!-- <link name="hand_link">
-        <visual>
-            <geometry>
-                <box size="${base_length} ${base_width} ${base_height}" />
-            </geometry>
-            <origin xyz="0 0 ${base_height / 2.0}" rpy="0 0 0" />
-            <material name="green" />
-        </visual>
-        <collision>
-            <geometry>
-                <box size="${base_length} ${base_width} ${base_height}" />
-            </geometry>
-            <origin xyz="0 0 ${base_height / 2.0}" rpy="0 0 0" />
-        </collision>
-        <xacro:box_inertia m="5.0" l="${2*base_length}" w="${2*base_width}" h="${2*base_height}"
-                           xyz="0 0 ${base_height}" rpy="0 0 0" />
-    </link> -->
-    <joint name= "base_joint" type ="fixed">
-        <parent link = "base_footprint" />
-        <child link = "box_link" />
-        <origin xyz = "0 0 0" rpy = "0 0 0" />
-    </joint>
-    <joint name= "base_joint" type ="fixed">
-        <parent link = "box_link" />
-        <child link = "forearm_link" />
-        <origin xyz="0 0 ${box_height/2.0}" rpy="0 0 0" />
-        <axis xyz = "1 0 0" />
-    </joint>
-</robot>
+/home/sambhav/ros2_ws/src/my_robot_description/urdf/robotic_arm.xacro

File: src/my_robot_description/urdf/common_properties.xacro (robot description, xacro)
@@ -6,4 +6,10 @@
     <material name="grey">
         <color rgba="0.5 0.5 0.5 1" />
+    </material>
+    <material name="orange">
+        <color rgba="0.98 0.4 0.05 1" />
+    </material>
+    <material name="yellow">
+        <color rgba="1 1 0 1" />
     </material>
     <xacro:macro name="box_inertia" params="m l w h xyz rpy">
@@ -34,3 +40,12 @@
         </inertial>
     </xacro:macro>
+    <xacro:macro name="rod_inertia" params="m r h xyz rpy">
+        <inertial>
+            <origin xyz="${xyz}" rpy="${rpy}" />
+            <mass value="${m}" />
+            <inertia ixx="${(m/3) * (h*h)}" ixy="0" ixz="0"
+                     iyy="0"                iyz="0"
+                     izz="${(m/3) * (h*h)}" />
+        </inertial>
+    </xacro:macro>
 </robot>

File: src/my_robot_description/urdf/my_robot.urdf.xacro (robot description, xacro)
@@ -3,4 +3,5 @@
     <xacro:include filename="common_properties.xacro" />
     <xacro:include filename="mobile_base.xacro" />
+    <xacro:include filename="robotic_arm.xacro" />
     <xacro:include filename="mobile_base_gazebo.xacro" />
     <xacro:include filename="camera.xacro" />

File: src/my_robot_description/urdf/robotic_arm.xacro (robot description, xacro)
@@ -1,5 +1,4 @@
 <?xml version = "1.0"?>
 <robot xmlns:xacro="http://www.ros.org/wiki/xacro">
-    <xacro:include filename="common_properties.xacro" />
     <xacro:property name="forearm_length" value = "0.3" />
     <xacro:property name="forearm_radius" value = "0.02" />
@@ -9,6 +8,7 @@
     <xacro:property name="box_width" value = "0.1" />
     <xacro:property name="box_height" value = "0.02" />
-    <link name = "base_footprint" />
-    <link name="box_link">
+<!--
+    <link name = "base_footprint" /> -->
+    <link name="arm_base_link">
         <visual>
             <geometry>
@@ -16,5 +16,5 @@
             </geometry>
             <origin xyz="0 0 ${box_height/2.0}" rpy="0 0 0" />
-            <material name="green" />
+            <material name="orange" />
         </visual>
         <collision>
@@ -32,6 +32,6 @@
                 <cylinder radius = "${forearm_radius}" length = "${forearm_length}" />
             </geometry>
-            <origin xyz="0 0 0" rpy="0 0 0" />
-            <material name="green" />
+            <origin xyz="0 0 ${forearm_length/2.0}" rpy="0 0 0" />
+            <material name="yellow" />
         </visual>
         <collision>
@@ -41,34 +41,42 @@
             <origin xyz="0 0 0" rpy="0 0 0" />
         </collision>
-        <xacro:cylinder_inertia m="1.0" r="${2*forearm_radius}" h="${2*forearm_length}"
+        <xacro:rod_inertia m="0.3" r="${2*forearm_radius}" h="${2*forearm_length}"
                        xyz="0 0 0" rpy="$0 0 0" />
     </link>
-    <!-- <link name="hand_link">
+    <link name="hand_link">
         <visual>
             <geometry>
-                <box size="${base_length} ${base_width} ${base_height}" />
+                <cylinder radius = "${hand_radius}" length = "${hand_length}" />
             </geometry>
-            <origin xyz="0 0 ${base_height / 2.0}" rpy="0 0 0" />
-            <material name="green" />
+            <origin xyz="0 0 ${hand_length/2.0}" rpy="0 0 0" />
+            <material name="orange" />
         </visual>
         <collision>
             <geometry>
-                <box size="${base_length} ${base_width} ${base_height}" />
+                <cylinder radius = "${hand_radius}" length = "${hand_length}" />
             </geometry>
-            <origin xyz="0 0 ${base_height / 2.0}" rpy="0 0 0" />
+            <origin xyz="0 0 ${hand_length/2.0}" rpy="0 0 0" />
         </collision>
-        <xacro:box_inertia m="5.0" l="${2*base_length}" w="${2*base_width}" h="${2*base_height}"
-                           xyz="0 0 ${base_height}" rpy="0 0 0" />
-    </link> -->
-    <joint name= "base_joint" type ="fixed">
-        <parent link = "base_footprint" />
-        <child link = "box_link" />
-        <origin xyz = "0 0 0" rpy = "0 0 0" />
+        <xacro:rod_inertia m="0.3" r="${2*hand_radius}" h="${2*hand_length}"
+                           xyz="0 0 0" rpy="0 0 0" />
+    </link>
+    <!-- <joint name= "base_arm_base_joint" type ="fixed">
+        <parent link = "base_link" />
+        <child link = "arm_base_link" />
+        <origin xyz = "0 0 ${base_height}" rpy = "0 0 0" />
+    </joint> -->
+    <joint name= "arm_base_forearm_joint" type ="revolute">
+        <parent link = "arm_base_link" />
+        <child link = "forearm_link" />
+        <origin xyz="0 0 ${box_height}" rpy="0 0 0" />
+        <axis xyz = "0 1 0" />
+        <limit lower = "0" upper = "${pi/2.0}" effort = "100" velocity = "100" />
     </joint>
-    <joint name= "base_joint" type ="fixed">
-        <parent link = "box_link" />
-        <child link = "forearm_link" />
-        <origin xyz="0 0 ${box_height/2.0}" rpy="0 0 0" />
-        <axis xyz = "1 0 0" />
+    <joint name= "forearm_hand_joint" type ="revolute">
+        <parent link = "forearm_link" />
+        <child link = "hand_link" />
+        <origin xyz="0 0 ${hand_length}" rpy="0 0 0" />
+        <axis xyz = "0 1 0" />
+        <limit lower = "0" upper = "${pi/2.0}" effort = "100" velocity = "100" />
     </joint>
 </robot>
