Commit message: action server

File: src/my_robot_description/urdf/my_robot.urdf.xacro (robot description, xacro)
@@ -3,7 +3,13 @@
     <xacro:include filename="common_properties.xacro" />
     <xacro:include filename="mobile_base.xacro" />
+    <xacro:include filename="mobile_base_gazebo.xacro" />
     <xacro:include filename="robotic_arm.xacro" />
-    <xacro:include filename="mobile_base_gazebo.xacro" />
-    <xacro:include filename="camera.xacro" />
+    <xacro:include filename="robotic_arm_gazebo.xacro" />
+    <joint name= "base_arm_base_joint" type ="fixed">
+        <parent link = "base_link" />
+        <child link = "arm_base_link" />
+        <origin xyz = "${base_length/4.0} 0 ${base_height}" rpy = "0 0 0" />
+    </joint>
+    <!-- <xacro:include filename="camera.xacro" /> -->
 </robot>
     <!-- <link name="right_wheel_link">

File: src/my_robot_description/urdf/robotic_arm.xacro (robot description, xacro)
@@ -39,8 +39,8 @@
                 <cylinder radius="${forearm_radius}" length="${forearm_length}" />
             </geometry>
-            <origin xyz="0 0 0" rpy="0 0 0" />
+            <origin xyz="0 0 ${forearm_length/2.0}" rpy="0 0 0" />
         </collision>
         <xacro:rod_inertia m="0.3" r="${2*forearm_radius}" h="${2*forearm_length}"
-                       xyz="0 0 0" rpy="$0 0 0" />
+                           xyz="0 0 ${forearm_length/2.0}" rpy="0 0 0" />
     </link>
     <link name="hand_link">
@@ -59,11 +59,6 @@
         </collision>
         <xacro:rod_inertia m="0.3" r="${2*hand_radius}" h="${2*hand_length}"
-                           xyz="0 0 0" rpy="0 0 0" />
+                                   xyz="0 0 ${hand_length/2.0}" rpy="0 0 0" />
     </link>
-    <!-- <joint name= "base_arm_base_joint" type ="fixed">
-        <parent link = "base_link" />
-        <child link = "arm_base_link" />
-        <origin xyz = "0 0 ${base_height}" rpy = "0 0 0" />
-    </joint> -->
     <joint name= "arm_base_forearm_joint" type ="revolute">
         <parent link = "arm_base_link" />
@@ -72,11 +67,13 @@
         <axis xyz = "0 1 0" />
         <limit lower = "0" upper = "${pi/2.0}" effort = "100" velocity = "100" />
+        <dynamics friction="0.05" damping="0.1" />
     </joint>
     <joint name= "forearm_hand_joint" type ="revolute">
         <parent link = "forearm_link" />
         <child link = "hand_link" />
-        <origin xyz="0 0 ${hand_length}" rpy="0 0 0" />
+        <origin xyz="0 0 ${forearm_length}" rpy="0 0 0" />
         <axis xyz = "0 1 0" />
         <limit lower = "0" upper = "${pi/2.0}" effort = "100" velocity = "100" />
+        <dynamics friction="0.05" damping="0.1" />
     </joint>
 </robot>

File: src/my_robot_description/urdf/robotic_arm_gazebo.xacro (robot description, xacro)
@@ -10,3 +10,20 @@
         <material>Gazebo/Orange</material>
     </gazebo>
+    <gazebo>
+        <plugin name="joint_state_publisher_controller"
+                filename="libgazebo_ros_joint_state_publisher.so">
+      <!-- Update rate in Hertz -->
+      <update_rate>10</update_rate>
+      <!-- Name of joints in the model whose states will be published. -->
+      <joint_name>arm_base_forearm_joint</joint_name>
+      <joint_name>forearm_hand_joint</joint_name>
+    </plugin>
+    </gazebo>
+    <gazebo>
+        <plugin name="joint_pose_trajectory_controller"
+                filename="libgazebo_ros_joint_pose_trajectory.so">
+      <!-- Update rate in Hz -->
+      <update_rate>2</update_rate>
+    </plugin>
+    </gazebo>
 </robot>
