Commit message: stopped working

File: src/install/my_robot_description/share/my_robot_description/urdf/common_properties.xacro (robot description, xacro)
@@ -7,3 +7,45 @@
         <color rgba="0.5 0.5 0.5 1" />
     </material>
+    <material name="orange">
+        <color rgba="0.98 0.4 0.05 1" />
+    </material>
+    <material name="yellow">
+        <color rgba="1 1 0 1" />
+    </material>
+    <xacro:macro name="box_inertia" params="m l w h xyz rpy">
+        <inertial>
+            <origin xyz="${xyz}" rpy="${rpy}" />
+            <mass value="${m}" />
+            <inertia ixx="${(m/12.0) * (h*h + l*l)}" ixy="0" ixz="0"
+                     iyy="${(m/12.0) * (w*w + l*l)}" iyz="0"
+                     izz="${(m/12.0) * (w*w + h*h)}" />
+        </inertial>
+    </xacro:macro>
+    <xacro:macro name="sphere_inertia" params="m r xyz rpy">
+        <inertial>
+            <origin xyz="${xyz}" rpy="${rpy}" />
+            <mass value="${m}" />
+            <inertia ixx="${(m * 2.0/5.0) * (r*r)}" ixy="0" ixz="0"
+                     iyy="${(m * 2.0/5.0) * (r*r)}"  iyz="0"
+                     izz="${(m * 2.0/5.0) * (r*r)}" />
+        </inertial>
+    </xacro:macro>
+    <xacro:macro name="cylinder_inertia" params="m r h xyz rpy">
+        <inertial>
+            <origin xyz="${xyz}" rpy="${rpy}" />
+            <mass value="${m}" />
+            <inertia ixx="${(m/12) * (3*r*r + h*h)}" ixy="0" ixz="0"
+                     iyy="${(m/12) * (3*r*r + h*h)}" iyz="0"
+                     izz="${(m/12) * (3*r*r + h*h)}" />
+        </inertial>
+    </xacro:macro>
+    <xacro:macro name="rod_inertia" params="m r h xyz rpy">
+        <inertial>
+            <origin xyz="${xyz}" rpy="${rpy}" />
+            <mass value="${m}" />
+            <inertia ixx="${(m/3) * (h*h)}" ixy="0" ixz="0"
+                     iyy="0"                iyz="0"
+                     izz="${(m/3) * (h*h)}" />
+        </inertial>
+    </xacro:macro>
 </robot>

File: src/install/my_robot_description/share/my_robot_description/urdf/mobile_base.xacro (robot description, xacro)
@@ -12,7 +12,15 @@
                 <box size="${base_length} ${base_width} ${base_height}" />
             </geometry>
-            <origin xyz="0 0 0.1" rpy="0 0 0" />
+            <origin xyz="0 0 ${base_height / 2.0}" rpy="0 0 0" />
             <material name="green" />
         </visual>
+        <collision>
+            <geometry>
+                <box size="${base_length} ${base_width} ${base_height}" />
+            </geometry>
+            <origin xyz="0 0 ${base_height / 2.0}" rpy="0 0 0" />
+        </collision>
+        <xacro:box_inertia m="5.0" l="${2*base_length}" w="${2*base_width}" h="${2*base_height}"
+                           xyz="0 0 ${base_height}" rpy="0 0 0" />
     </link>
     <xacro:macro name="wheel_link" params="prefix">
@@ -25,4 +33,12 @@
                 <material name="grey" />
             </visual>
+            <collision>
+                <geometry>
+                    <cylinder radius="${wheel_radius}" length="${wheel_length}" />
+                </geometry>
+                <origin xyz="0 0 0" rpy="${pi / 2.0} 0 0" />
+            </collision>
+            <xacro:cylinder_inertia m="1.0" r="${2*wheel_radius}" h="${2*wheel_length}"
+                           xyz="0 0 0" rpy="${pi / 2.0} 0 0" />
         </link>
     </xacro:macro>
@@ -32,9 +48,17 @@
         <visual>
             <geometry>
-                <sphere radius="0.05"/>
+                <sphere radius="${wheel_radius/2.0}"/>
             </geometry>
             <origin xyz="0 0 0" rpy="0 0 0" />
             <material name="grey" />
         </visual>
+        <collision>
+            <geometry>
+                <sphere radius="${wheel_radius/2.0}"/>
+            </geometry>
+            <origin xyz="0 0 0" rpy="0 0 0" />
+        </collision>
+        <xacro:sphere_inertia m="0.5" r="${2*wheel_radius / 2.0}"
+                           xyz="0 0 0" rpy="0 0 0" />
     </link>
     <joint name="base_joint" type="fixed">
@@ -46,5 +70,5 @@
         <parent link="base_link" />
         <child link="right_wheel_link" />
-        <origin xyz="${-base_length / 4.0} ${(-base_width / 2.0) + (-wheel_radius / 2.0)} 0" rpy="0 0 0" />
+        <origin xyz="${-base_length / 4.0} ${(base_width / 2.0) + (wheel_length / 2.0)} 0" rpy="0 0 0" />
         <axis xyz="0 1 0" />
     </joint>
@@ -52,5 +76,5 @@
         <parent link="base_link" />
         <child link="left_wheel_link" />
-        <origin xyz="${-base_length / 4.0} ${(base_width / 2.0) + (wheel_radius / 2.0)} 0" rpy="0 0 0" />
+        <origin xyz="${-base_length / 4.0} ${(-base_width / 2.0) + (-wheel_length / 2.0)} 0" rpy="0 0 0" />
         <axis xyz="0 1 0" />
     </joint>

File: src/install/my_robot_description/share/my_robot_description/urdf/my_robot.urdf.xacro (robot description, xacro)
@@ -3,4 +3,13 @@
     <xacro:include filename="common_properties.xacro" />
     <xacro:include filename="mobile_base.xacro" />
+    <xacro:include filename="mobile_base_gazebo.xacro" />
+    <xacro:include filename="robotic_arm.xacro" />
+    <xacro:include filename="robotic_arm_gazebo.xacro" />
+    <joint name= "base_arm_base_joint" type ="fixed">
+        <parent link = "base_link" />
+        <child link = "arm_base_link" />
+        <origin xyz = "${base_length/4.0} 0 ${base_height}" rpy = "0 0 0" />
+    </joint>
+    <!-- <xacro:include filename="camera.xacro" /> -->
 </robot>
     <!-- <link name="right_wheel_link">
